File: Circuit/Schematics/Wifi.sch (EAGLE design)
At the start: 18 parts

Commit message: Wifi and mesh board crappy designed
Parts:
- removed E1: ANTENNATRACE-15.2MM, SparkFun-RF:ANTENNATRACE-15.2MM
- added U$3: ANTENNA2SMD, SparkFun-RF:ANTENNA2SMD
Connections:
- new net N$1: C1.2, U$3.SIGNAL
- new net VDD: C18.2, U$2.VCC
- net VCC: no longer C18.2, U$2.VCC
Changed lines of the file:
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@@
 <part name="JP1" library="adafruit" deviceset="PINHD-1X8" device="BIG"/>
 <part name="C1" library="SparkFun-Capacitors" deviceset="CAP" device="0402-CAP" value="5.6 pF"/>
-<part name="E1" library="SparkFun-RF" deviceset="ANTENNA" device="TRACE-15.2MM"/>
+<part name="U$3" library="SparkFun-RF" deviceset="ANTENNA2" device="SMD"/>
 </parts>
 <sheets>
@@
 <instance part="JP1" gate="G$1" x="213.36" y="106.68"/>
 <instance part="C1" gate="G$1" x="68.58" y="58.42" rot="R270"/>
-<instance part="E1" gate="G$1" x="48.26" y="71.12"/>
+<instance part="U$3" gate="G$1" x="60.96" y="63.5"/>
 </instances>
 <busses>
@@
 </net>
 <net name="VCC" class="0">
-<segment>
-<pinref part="P+1" gate="1" pin="VCC"/>
-<wire x1="228.6" y1="101.6" x2="228.6" y2="96.52" width="0.1524" layer="91"/>
-</segment>
 <segment>
 <pinref part="U$1" gate="G$1" pin="VDDA/30"/>
@@
 </segment>
 <segment>
-<pinref part="U$2" gate="G$1" pin="VCC"/>
-<wire x1="254" y1="53.34" x2="259.08" y2="53.34" width="0.1524" layer="91"/>
-<junction x="259.08" y="53.34"/>
-<wire x1="259.08" y1="53.34" x2="261.62" y2="53.34" width="0.1524" layer="91"/>
-<wire x1="259.08" y1="53.34" x2="259.08" y2="58.42" width="0.1524" layer="91"/>
-<pinref part="C18" gate="G$1" pin="2"/>
-</segment>
-<segment>
 <pinref part="JP1" gate="G$1" pin="2"/>
 <wire x1="210.82" y1="111.76" x2="203.2" y2="111.76" width="0.1524" layer="91"/>
@@
 </segment>
 </net>
+<net name="N$1" class="0">
+<segment>
+<pinref part="C1" gate="G$1" pin="2"/>
+<wire x1="66.04" y1="58.42" x2="60.96" y2="58.42" width="0.1524" layer="91"/>
+<pinref part="U$3" gate="G$1" pin="SIGNAL"/>
+</segment>
+</net>
+<net name="VDD" class="0">
+<segment>
+<pinref part="P+1" gate="1" pin="VCC"/>
+<wire x1="228.6" y1="101.6" x2="228.6" y2="96.52" width="0.1524" layer="91"/>
+</segment>
+<segment>
+<pinref part="U$2" gate="G$1" pin="VCC"/>
+<wire x1="254" y1="53.34" x2="259.08" y2="53.34" width="0.1524" layer="91"/>
+<junction x="259.08" y="53.34"/>
+<wire x1="259.08" y1="53.34" x2="261.62" y2="53.34" width="0.1524" layer="91"/>
+<wire x1="259.08" y1="53.34" x2="259.08" y2="58.42" width="0.1524" layer="91"/>
+<pinref part="C18" gate="G$1" pin="2"/>
+</segment>
+</net>
