File: Circuit/Schematics/Teensy.sch (EAGLE design)
At the start: 36 parts, among them Y1 16 MHz, Y2 32.768 kHz

Commit message: Teensy board designed, redesigning system components board and making hardware components consistent
Parts:
- C2, C3, C6: value (none) -> 0.1 uF
- renumbered F2 to FUSE
Connections:
- net N$17 renamed T_TX
- net N$21 renamed CE
- net N$34 renamed SCK
- net N$7 renamed T_RX
Changed lines of the file:
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@@
 <part name="U$3" library="Teensy_3_Series_Chip_v1.2" deviceset="MINI54TAN" device="DEFAULT"/>
 <part name="C1" library="SparkFun-Capacitors" deviceset="CAP_POL" device="1206" value="0.1uF"/>
-<part name="C2" library="SparkFun-Capacitors" deviceset="CAP_POL" device="1206"/>
-<part name="C3" library="SparkFun-Capacitors" deviceset="CAP_POL" device="1206"/>
+<part name="C2" library="SparkFun-Capacitors" deviceset="CAP_POL" device="1206" value="0.1 uF"/>
+<part name="C3" library="SparkFun-Capacitors" deviceset="CAP_POL" device="1206" value="0.1 uF"/>
 <part name="C4" library="SparkFun-Capacitors" deviceset="CAP_POL" device="1206" value="0.1uF"/>
 <part name="C5" library="SparkFun-Capacitors" deviceset="CAP_POL" device="1206" value="0.1uF"/>
-<part name="C6" library="SparkFun-Capacitors" deviceset="CAP_POL" device="1206"/>
+<part name="C6" library="SparkFun-Capacitors" deviceset="CAP_POL" device="1206" value="0.1 uF"/>
 <part name="GND-ISO3" library="SparkFun-Aesthetics" deviceset="GND-ISO" device=""/>
 <part name="GND-ISO4" library="SparkFun-Aesthetics" deviceset="GND-ISO" device=""/>
@@
 <part name="JP7" library="SparkFun-Connectors" deviceset="M02" device="LOCK"/>
 <part name="JP8" library="SparkFun-Connectors" deviceset="M02" device="LOCK"/>
-<part name="F2" library="SparkFun-PowerIC" deviceset="PTC" device="0603"/>
+<part name="FUSE" library="SparkFun-PowerIC" deviceset="PTC" device="0603"/>
 <part name="JP9" library="SparkFun-Connectors" deviceset="M09" device=""/>
 <part name="GPIO" library="SparkFun-Connectors" deviceset="M08" device="SILK_FEMALE_PTH"/>
@@
 <instance part="JP7" gate="G$1" x="223.52" y="119.38" rot="R180"/>
 <instance part="JP8" gate="G$1" x="223.52" y="104.14" rot="R180"/>
-<instance part="F2" gate="G$1" x="40.64" y="162.56" rot="R90"/>
+<instance part="FUSE" gate="G$1" x="40.64" y="162.56" rot="R90"/>
 <instance part="JP9" gate="G$1" x="210.82" y="137.16" rot="R180"/>
 <instance part="GPIO" gate="G$1" x="205.74" y="106.68" rot="R180"/>
@@
 <wire x1="40.64" y1="182.88" x2="86.36" y2="182.88" width="0.1524" layer="91"/>
 <junction x="86.36" y="182.88"/>
-<pinref part="F2" gate="G$1" pin="2"/>
+<pinref part="FUSE" gate="G$1" pin="2"/>
 </segment>
 </net>
@@
 </segment>
 </net>
-<net name="N$34" class="0">
+<net name="SCK" class="0">
 <segment>
 <pinref part="U$2" gate="G$1" pin="D13/SCK/LED"/>
@@
 <pinref part="JP1" gate="G$1" pin="VCC"/>
 <wire x1="25.4" y1="132.08" x2="17.78" y2="132.08" width="0.1524" layer="91"/>
-<pinref part="F2" gate="G$1" pin="1"/>
+<pinref part="FUSE" gate="G$1" pin="1"/>
 <wire x1="40.64" y1="154.94" x2="40.64" y2="157.48" width="0.1524" layer="91"/>
 </segment>
@@
 </segment>
 </net>
-<net name="N$7" class="0">
+<net name="T_RX" class="0">
 <segment>
 <pinref part="U$2" gate="G$1" pin="D0/RX1/TOUCH"/>
@@
 </segment>
 </net>
-<net name="N$17" class="0">
+<net name="T_TX" class="0">
 <segment>
 <pinref part="U$2" gate="G$1" pin="D1/TX1/TOUCH"/>
@@
 </segment>
 </net>
-<net name="N$21" class="0">
+<net name="CE" class="0">
 <segment>
 <pinref part="U$2" gate="G$1" pin="D9/RX2/PWM"/>
