File: Circuit/Schematics/top.sch (EAGLE design)
At the start: 36 parts, among them Y1 16 MHz, Y2 32.768 kHz

Commit message: P1 preliminary boards finished
Parts:
- removed C1, C4, C5, C7, C8, C9: 0.1uF, SparkFun-Capacitors:CAP_POL1206
- removed C10: 2.2uF, SparkFun-Capacitors:CAP_POL1206
- removed C2, C3, C6: 0.1 uF, SparkFun-Capacitors:CAP_POL1206
- added C11, C12, C13, C14, C15, C17, C18, C19, C20: .1 uF, SparkFun-Passives:CAP0603-CAP
- added C16: 2.2 uF, SparkFun-Passives:CAP0603-CAP
Connections:
- net 3.3V: now also C13.1, C14.1, C15.1, C16.1; no longer C10.+, C7.+, C8.+, C9.+
- net AGND: now also C17.2, C18.2, C19.2; no longer C4.-, C5.-, C6.-
- net GND-ISO: now also C11.1, C12.1, C13.2, C14.2, C15.2, C16.2, C20.2; no longer C1.-, C10.-, C2.-, C3.-, C7.-, C8.-, C9.-
- net N$1: now also C19.1; no longer C4.+
- net N$2: now also C12.2; no longer C1.+
- net N$4: now also C17.1; no longer C6.+
- net N$5: now also C18.1; no longer C5.+
- net N$63: now also C11.2; no longer C3.+
- net N$9: now also C20.1; no longer C2.+
